Commit message: Camera Mount Added

File: src/robo1/urdf/integration.urdf.xacro (robot description, xacro)
@@ -2,4 +2,5 @@
 <robot name ="robo1" xmlns:xacro="http://wiki.ros.org/xacro">
 	<xacro:include filename="$(find robo1)/urdf/robo1.urdf"/>
+	<xacro:include filename="$(find robo1)/urdf/camera.urdf"/>
 	<gazebo>
 		<plugin name="gazebo_ros_control" filename="libgazebo_ros_control.so">
@@ -9,3 +10,16 @@
 		</plugin>
 	</gazebo>
+	<joint
+    name="camera_joint"
+    type="fixed">
+    <origin
+      xyz="0 0 0"
+      rpy="0 0 0" />
+    <parent
+      link="camhold_link" />
+    <child
+      link="camera_link" />
+    <axis
+      xyz="0 0 0" />
+  </joint>
 </robot>

File: src/robo1/urdf/robo1.urdf (robot description, URDF)
Before this commit: robot robo1, 13 links, 12 joints
Joints:
- joint camhold_joint: origin xyz=-0.148 0 0.029 rpy=1.5708 0 0 -> xyz=-0.155 0.015 0.034 rpy=3.14159 0 0

Commit message: commented incomplete inputs to run temporarily

File: src/robo1/urdf/integration.urdf.xacro (robot description, xacro)
@@ -2,5 +2,5 @@
 <robot name ="robo1" xmlns:xacro="http://wiki.ros.org/xacro">
 	<xacro:include filename="$(find robo1)/urdf/robo1.urdf"/>
-	<xacro:include filename="$(find robo1)/urdf/camera.urdf"/>
+	<!--xacro:include filename="$(find robo1)/urdf/camera.urdf"/-->
 	<gazebo>
 		<plugin name="gazebo_ros_control" filename="libgazebo_ros_control.so">
@@ -10,5 +10,5 @@
 		</plugin>
 	</gazebo>
-	<joint
+	<!--joint
     name="camera_joint"
     type="fixed">
@@ -22,4 +22,4 @@
     <axis
       xyz="0 0 0" />
-  </joint>
+  </joint-->
 </robot>
