Commit message: ROS model with transmission added, working fine

File: src/robo1/urdf/robo1.urdf (robot description, URDF)
Before this commit: robot robo1, 13 links, 12 joints
Joints:
- joint castor1_joint: origin xyz=-0.145 0.01 0.06375 rpy=3.1416 -1.5708 0 -> xyz=-0.145 0.005 0.06375 rpy=3.1416 -1.5708 3.14159
- joint castor2_joint: origin xyz=-0.145 0.01 -0.06375 rpy=3.1416 -1.5708 0 -> xyz=-0.145 0.005 -0.06375 rpy=3.1416 -1.5708 3.14159

Commit message: added world

File: src/robo1/urdf/robo1.urdf (robot description, URDF)
Before this commit: robot robo1, 13 links, 12 joints
Links:
- link arduino_link: geometry collision mesh filename=$(find robo1)/meshes/arduino_link.STL; visual mesh filename=$(find robo1)/meshes/arduino_link.STL
- link base_link: geometry collision mesh filename=$(find robo1)/meshes/base_link.STL; visual mesh filename=$(find robo1)/meshes/base_link.STL
- link battery_link: geometry collision mesh filename=$(find robo1)/meshes/battery_link.STL; visual mesh filename=$(find robo1)/meshes/battery_link.STL
- link camhold_link: geometry collision mesh filename=$(find robo1)/meshes/camhold_link.STL; visual mesh filename=$(find robo1)/meshes/camhold_link.STL
- link castor1_link: geometry collision mesh filename=$(find robo1)/meshes/castor1_link.STL; visual mesh filename=$(find robo1)/meshes/castor1_link.STL
- link castor2_link: geometry collision mesh filename=$(find robo1)/meshes/castor2_link.STL; visual mesh filename=$(find robo1)/meshes/castor2_link.STL
- link motorL_link: geometry collision mesh filename=$(find robo1)/meshes/motorL_link.STL; visual mesh filename=$(find robo1)/meshes/motorL_link.STL
- link motorR_link: geometry collision mesh filename=$(find robo1)/meshes/motorR_link.STL; visual mesh filename=$(find robo1)/meshes/motorR_link.STL
- link rpi_link: geometry collision mesh filename=$(find robo1)/meshes/rpi_link.STL; visual mesh filename=$(find robo1)/meshes/rpi_link.STL
- link top_link: geometry collision mesh filename=$(find robo1)/meshes/top_link.STL; visual mesh filename=$(find robo1)/meshes/top_link.STL
- link wheelL_link: geometry collision mesh filename=$(find robo1)/meshes/wheelL_link.STL; visual mesh filename=$(find robo1)/meshes/wheelL_link.STL
- link wheelR_link: geometry collision mesh filename=$(find robo1)/meshes/wheelR_link.STL; visual mesh filename=$(find robo1)/meshes/wheelR_link.STL
Joints:
- joint base_to_dummy_joint: origin xyz=0 0 0.1 rpy=-1.5707963267 0 0 -> xyz=0 0 0.1 rpy=-1.5707963267 0 -1.57079

Commit message: Simulation files changed from bot files, p2p plan

File: src/robo1/urdf/robo1.urdf (robot description, URDF)
Before this commit: robot robo1, 13 links, 12 joints
Links:
- link base_link: mass 0.45001 -> 4.5001
- link wheelL_link: mass 0.056366 -> 0.56366
- link wheelR_link: mass 0.056366 -> 0.56366

Commit message: smooth trajec generator changes

File: src/robo1/urdf/robo1.urdf (robot description, URDF)
Before this commit: robot robo1, 13 links, 12 joints
Links:
- link arduino_link: geometry collision mesh filename=package://robo1/meshes/arduino_link.STL; visual mesh filename=package://robo1/meshes/arduino_link.STL
- link base_link: geometry collision mesh filename=package://robo1/meshes/base_link.STL; visual mesh filename=package://robo1/meshes/base_link.STL
- link battery_link: geometry collision mesh filename=package://robo1/meshes/battery_link.STL; visual mesh filename=package://robo1/meshes/battery_link.STL
- link camhold_link: geometry collision mesh filename=package://robo1/meshes/camhold_link.STL; visual mesh filename=package://robo1/meshes/camhold_link.STL
- link castor1_link: geometry collision mesh filename=package://robo1/meshes/castor1_link.STL; visual mesh filename=package://robo1/meshes/castor1_link.STL
- link castor2_link: geometry collision mesh filename=package://robo1/meshes/castor2_link.STL; visual mesh filename=package://robo1/meshes/castor2_link.STL
- link motorL_link: geometry collision mesh filename=package://robo1/meshes/motorL_link.STL; visual mesh filename=package://robo1/meshes/motorL_link.STL
- link motorR_link: geometry collision mesh filename=package://robo1/meshes/motorR_link.STL; visual mesh filename=package://robo1/meshes/motorR_link.STL
- link rpi_link: geometry collision mesh filename=package://robo1/meshes/rpi_link.STL; visual mesh filename=package://robo1/meshes/rpi_link.STL
- link top_link: geometry collision mesh filename=package://robo1/meshes/top_link.STL; visual mesh filename=package://robo1/meshes/top_link.STL
- link wheelL_link: geometry collision mesh filename=package://robo1/meshes/wheelL_link.STL; visual mesh filename=package://robo1/meshes/wheelL_link.STL
- link wheelR_link: geometry collision mesh filename=package://robo1/meshes/wheelR_link.STL; visual mesh filename=package://robo1/meshes/wheelR_link.STL

Commit message: Rviz visualization

File: src/robo1/urdf/robo1.urdf (robot description, URDF)
Before this commit: robot robo1, 13 links, 12 joints
Joints:
- joint base_to_dummy_joint: origin xyz=0 0 0.1 rpy=-1.5707963267 0 -1.57079 -> xyz=0 0 0.035 rpy=-1.5707963267 0 -3.14159

Commit message: added RVIZ config and launch files

File: src/robo1/urdf/robo1.urdf (robot description, URDF)
Before this commit: robot robo1, 13 links, 12 joints
Joints:
- joint base_to_dummy_joint: origin xyz=0 0 0.035 rpy=-1.5707963267 0 -3.14159 -> xyz=0 0 0.035 rpy=-1.5707963267 0 -1.5707963267
- joint wheelL_joint: type continuous -> fixed
- joint wheelR_joint: type continuous -> fixed
